File: Nunam_Cell_Harness.kicad_pcb (KiCad board)
At the start: 2 copper layers, 598 x 62.4 mm, 17 parts, among them J1 Conn_01x14, J10 CELL_7+/10+, J11 CELL_8+/9+, J12 NTC1_A, J13 NTC1_B, J14 NTC2_A, J15 NTC2_B, J2 BATT-/NC, J3 CELL_1-/BATT+, J4 CELL_1+/16+, J5 CELL_2+/15+, J6 CELL_3+/14+, J7 CELL_4+/13+, J8 CELL_5+/12+, J9 CELL_6+/11+

Commit message: Removed signature and PCB fabricated
Other:
- board text removed: "Vaibhav Khatri"
Changed lines of the file:
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@@
 		(tags "connector JST XH horizontal")
 		(property "Reference" "J1"
-			(at 16.25 -3.51 90)
+			(at 15.95 -2.5 90)
 			(layer "F.SilkS")
 			(effects
@@
 		(layer "Edge.Cuts")
 	)
-	(gr_text "Vaibhav\nKhatri"
-		(at 742.499999 355.899999 0)
-		(layer "B.Cu")
-		(effects
-			(font
-				(size 1.5 1.5)
-				(thickness 0.3)
-				(bold yes)
-			)
-			(justify left bottom mirror)
-		)
-	)
 	(gr_text "Fabrication Details:\n1. PCB shall have a Tg of 130C\n2. PCB material: FR4\n3. PCB thickness: 1.6mm\n4. PCB finish: HASL\n5. Board layers: 2\n6. Copper thickness: 35um"
 		(at 147.999999 288.899999 0)
@@
 	)
 	(zone
-		(net "Net-(J1-Pin_2)")
+		(net "Net-(J1-Pin_12)")
 		(layer "F.Cu")
 		(hatch none 0.1)
-		(priority 30006)
+		(priority 30009)
 		(attr
 			(teardrop
@@
 		(polygon
 			(pts
-				(xy 335.824999 309.999999) (xy 336.174999 309.999999) (xy 336.999999 308.999999) (xy 335.999999 307.498999)
-				(xy 334.999999 308.999999)
+				(xy 263.174999 359.399999) (xy 262.824999 359.399999) (xy 261.999999 360.399999) (xy 262.999999 361.900999)
+				(xy 263.999999 360.399999)
 			)
 		)
 	)
 	(zone
-		(net "Net-(J1-Pin_4)")
+		(net "Net-(J1-Pin_3)")
 		(layer "F.Cu")
 		(hatch none 0.1)
-		(priority 30008)
+		(priority 30013)
 		(attr
 			(teardrop
@@
 		(polygon
 			(pts
-				(xy 627.824999 309.999999) (xy 628.174999 309.999999) (xy 628.999999 308.999999) (xy 627.999999 307.498999)
-				(xy 626.999999 308.999999)
+				(xy 481.824999 309.999999) (xy 482.174999 309.999999) (xy 482.999999 308.999999) (xy 481.999999 307.498999)
+				(xy 480.999999 308.999999)
 			)
 		)
 	)
 	(zone
-		(net "Net-(J1-Pin_6)")
+		(net "Net-(J1-Pin_13)")
 		(layer "F.Cu")
 		(hatch none 0.1)
-		(priority 30003)
+		(priority 30001)
 		(attr
 			(teardrop
@@
 		(polygon
 			(pts
-				(xy 215.499999 336.524999) (xy 215.499999 336.874999) (xy 216.499999 337.699999) (xy 218.000999 336.699999)
-				(xy 216.499999 335.699999)
+				(xy 190.174999 359.399999) (xy 189.824999 359.399999) (xy 188.999999 360.399999) (xy 189.999999 361.900999)
+				(xy 190.999999 360.399999)
 			)
 		)
 	)
 	(zone
-		(net "Net-(J1-Pin_10)")
+		(net "Net-(J1-Pin_14)")
 		(layer "F.Cu")
 		(hatch none 0.1)
-		(priority 30002)
+		(priority 30005)
 		(attr
 			(teardrop
@@
 		(polygon
 			(pts
-				(xy 555.174999 359.399999) (xy 554.824999 359.399999) (xy 553.999999 360.399999) (xy 554.999999 361.900999)
-				(xy 555.999999 360.399999)
+				(xy 176 353.724999) (xy 176 354.074999) (xy 177 354.899999) (xy 178.501 353.899999) (xy 177 352.899999)
 			)
 		)
@@
 	)
 	(zone
-		(net "Net-(J1-Pin_14)")
+		(net "Net-(J1-Pin_7)")
 		(layer "F.Cu")
 		(hatch none 0.1)
-		(priority 30005)
+		(priority 30011)
 		(attr
 			(teardrop
@@
 		(polygon
 			(pts
-				(xy 176 353.724999) (xy 176 354.074999) (xy 177 354.899999) (xy 178.501 353.899999) (xy 177 352.899999)
+				(xy 730.999999 332.524999) (xy 730.999999 332.874999) (xy 731.999999 333.699999) (xy 733.500999 332.699999)
+				(xy 731.999999 331.699999)
 			)
 		)
@@
 	)
 	(zone
-		(net "Net-(J1-Pin_7)")
+		(net "Net-(J1-Pin_9)")
 		(layer "F.Cu")
 		(hatch none 0.1)
-		(priority 30011)
+		(priority 30000)
 		(attr
 			(teardrop
@@
 		(polygon
 			(pts
-				(xy 730.999999 332.524999) (xy 730.999999 332.874999) (xy 731.999999 333.699999) (xy 733.500999 332.699999)
-				(xy 731.999999 331.699999)
+				(xy 701.174999 359.399999) (xy 700.824999 359.399999) (xy 699.999999 360.399999) (xy 700.999999 361.900999)
+				(xy 701.999999 360.399999)
 			)
 		)
 	)
 	(zone
-		(net "Net-(J1-Pin_13)")
+		(net "Net-(J1-Pin_10)")
 		(layer "F.Cu")
 		(hatch none 0.1)
-		(priority 30001)
+		(priority 30002)
 		(attr
 			(teardrop
@@
 		(polygon
 			(pts
-				(xy 190.174999 359.399999) (xy 189.824999 359.399999) (xy 188.999999 360.399999) (xy 189.999999 361.900999)
-				(xy 190.999999 360.399999)
+				(xy 555.174999 359.399999) (xy 554.824999 359.399999) (xy 553.999999 360.399999) (xy 554.999999 361.900999)
+				(xy 555.999999 360.399999)
 			)
 		)
 	)
 	(zone
-		(net "Net-(J1-Pin_9)")
+		(net "Net-(J1-Pin_6)")
 		(layer "F.Cu")
 		(hatch none 0.1)
-		(priority 30000)
+		(priority 30003)
 		(attr
 			(teardrop
@@
 		(polygon
 			(pts
-				(xy 701.174999 359.399999) (xy 700.824999 359.399999) (xy 699.999999 360.399999) (xy 700.999999 361.900999)
-				(xy 701.999999 360.399999)
+				(xy 215.499999 336.524999) (xy 215.499999 336.874999) (xy 216.499999 337.699999) (xy 218.000999 336.699999)
+				(xy 216.499999 335.699999)
 			)
 		)
 	)
 	(zone
-		(net "Net-(J1-Pin_12)")
+		(net "Net-(J1-Pin_11)")
 		(layer "F.Cu")
 		(hatch none 0.1)
-		(priority 30009)
+		(priority 30004)
 		(attr
 			(teardrop
@@
 		(polygon
 			(pts
-				(xy 263.174999 359.399999) (xy 262.824999 359.399999) (xy 261.999999 360.399999) (xy 262.999999 361.900999)
-				(xy 263.999999 360.399999)
+				(xy 409.174999 359.399999) (xy 408.824999 359.399999) (xy 407.999999 360.399999) (xy 408.999999 361.900999)
+				(xy 409.999999 360.399999)
 			)
 		)
 	)
 	(zone
-		(net "Net-(J1-Pin_3)")
+		(net "Net-(J1-Pin_4)")
 		(layer "F.Cu")
 		(hatch none 0.1)
-		(priority 30013)
+		(priority 30008)
 		(attr
 			(teardrop
@@
 		(polygon
 			(pts
-				(xy 481.824999 309.999999) (xy 482.174999 309.999999) (xy 482.999999 308.999999) (xy 481.999999 307.498999)
-				(xy 480.999999 308.999999)
+				(xy 627.824999 309.999999) (xy 628.174999 309.999999) (xy 628.999999 308.999999) (xy 627.999999 307.498999)
+				(xy 626.999999 308.999999)
 			)
 		)
 	)
 	(zone
-		(net "Net-(J1-Pin_8)")
+		(net "Net-(J1-Pin_2)")
 		(layer "F.Cu")
 		(hatch none 0.1)
-		(priority 30010)
+		(priority 30006)
 		(attr
 			(teardrop
@@
 		(polygon
 			(pts
-				(xy 730.999999 336.524999) (xy 730.999999 336.874999) (xy 731.999999 337.699999) (xy 733.500999 336.699999)
-				(xy 731.999999 335.699999)
+				(xy 335.824999 309.999999) (xy 336.174999 309.999999) (xy 336.999999 308.999999) (xy 335.999999 307.498999)
+				(xy 334.999999 308.999999)
 			)
 		)
 	)
 	(zone
-		(net "Net-(J1-Pin_11)")
+		(net "Net-(J1-Pin_8)")
 		(layer "F.Cu")
 		(hatch none 0.1)
-		(priority 30004)
+		(priority 30010)
 		(attr
 			(teardrop
@@
 		(polygon
 			(pts
-				(xy 409.174999 359.399999) (xy 408.824999 359.399999) (xy 407.999999 360.399999) (xy 408.999999 361.900999)
-				(xy 409.999999 360.399999)
+				(xy 730.999999 336.524999) (xy 730.999999 336.874999) (xy 731.999999 337.699999) (xy 733.500999 336.699999)
+				(xy 731.999999 335.699999)
 			)
 		)
